File: ratgdo-esp32c6-mini.kicad_sch (KiCad schematic)
At the start: 29 parts, among them J1 USB_C_Receptacle_USB2.0_14P, J2 Screw_Terminal_01x03, Q1 2N7002, Q2 AO3400A, SW1 RESET, SW2 BOOTSEL, U1 ESP32-C6-MINI-1/U, U2 RS3236-3.3YF5, U3 USBLC6-2SC6

Commit message: add footprint & LCSC PN
Parts:
- C1, C3: footprint (none) -> Capacitor_SMD:C_0805_2012Metric; LCSC PN (none) -> C116352
- C2: footprint (none) -> Capacitor_SMD:C_0805_2012Metric; LCSC PN (none) -> C1710
- C4: renamed from C5; footprint (none) -> Capacitor_SMD:C_0805_2012Metric; LCSC PN (none) -> C116352
- D1: footprint (none) -> LED_SMD:LED_0805_2012Metric; LCSC PN (none) -> C84260
- D2: footprint (none) -> LED_SMD:LED_0805_2012Metric; LCSC PN (none) -> C84256
- J1: footprint (none) -> Connector_USB:USB_C_Receptacle_G-Switch_GT-USB-7010ASV; LCSC PN (none) -> C2765186
- J2: footprint (none) -> TerminalBlock_CUI:TerminalBlock_CUI_TB007-508-03_1x03_P5.08mm_Horizontal; LCSC PN (none) -> C72334
- Q1: LCSC PN (none) -> C81445
- Q2: LCSC PN (none) -> C347475
- R1, R2: value 5.1k -> 5.1K; footprint (none) -> Resistor_SMD:R_0805_2012Metric; LCSC PN (none) -> C27834
- R10, R9: footprint (none) -> Resistor_SMD:R_0805_2012Metric; LCSC PN (none) -> C17513
- R11, R14: footprint (none) -> Resistor_SMD:R_0805_2012Metric; LCSC PN (none) -> C17414
- R12, R13, R5, R7, R8: value 10k -> 10K; footprint Resistor_SMD:R_0805_2012Metric_Pad1.20x1.40mm_HandSolder -> Resistor_SMD:R_0805_2012Metric; LCSC PN (none) -> C17414
- R3, R4: footprint (none) -> Resistor_SMD:R_0805_2012Metric; LCSC PN (none) -> C25295
- R6: value 1k -> 1K; footprint Resistor_SMD:R_0805_2012Metric_Pad1.20x1.40mm_HandSolder -> Resistor_SMD:R_0805_2012Metric; LCSC PN (none) -> C17513
- SW1, SW2: footprint (none) -> Button_Switch_SMD:SW_Push_SPST_NO_Alps_SKRK; LCSC PN (none) -> C720477
- U1: renamed from U3; LCSC PN (none) -> C7519
- U2: renamed from U1; LCSC PN (none) -> C5736265
- U3: renamed from U2; LCSC PN (none) -> C379349

Commit message: replace screw terminal with connector
Parts:
- removed J2: Screw_Terminal_01x03, TerminalBlock_CUI:TerminalBlock_CUI_TB007-508-03_1x03_P5.08mm_Horizontal, symbol Connector:Screw_Terminal_01x03
- added J2: Conn_01x03, LCSC:CONN-SMD_3P-P2.50_HX-2.54-3P-WT, symbol Connector_Generic:Conn_01x03
Connections:
- net BLK/OBST: now also J2.1 (Pin_1)
- net GND: now also J2.3 (Pin_3)
- net RED/CTRL: now also J2.2 (Pin_2)
Changed lines of the file:
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@@
-	)
-	(symbol
-		(lib_id "Connector:Screw_Terminal_01x03")
-		(at 247.65 58.42 0)
-		(unit 1)
-		(body_style 1)
-		(exclude_from_sim no)
-		(in_bom yes)
-		(on_board yes)
-		(in_pos_files yes)
-		(dnp no)
-		(property "Reference" "J2"
-			(at 247.65 50.8 0)
-			(show_name no)
-			(do_not_autoplace no)
-			(effects
-				(font
-					(size 1.27 1.27)
-				)
-				(justify left)
-			)
-		)
-		(property "Value" "Screw_Terminal_01x03"
-			(at 235.458 52.832 0)
-			(show_name no)
-			(do_not_autoplace no)
-			(effects
-				(font
-					(size 1.27 1.27)
-				)
-				(justify left)
-			)
-		)
-		(property "Footprint" "TerminalBlock_CUI:TerminalBlock_CUI_TB007-508-03_1x03_P5.08mm_Horizontal"
-			(at 247.65 58.42 0)
-			(hide yes)
-			(show_name no)
-			(do_not_autoplace no)
-			(effects
-				(font
-					(size 1.27 1.27)
-				)
-			)
-		)
-		(property "Datasheet" ""
-			(at 247.65 58.42 0)
-			(hide yes)
-			(show_name no)
-			(do_not_autoplace no)
-			(effects
-				(font
-					(size 1.27 1.27)
-				)
-			)
-		)
-		(property "Description" "Generic screw terminal, single row, 01x03, script generated (kicad-library-utils/schlib/autogen/connector/)"
-			(at 247.65 58.42 0)
-			(hide yes)
-			(show_name no)
-			(do_not_autoplace no)
-			(effects
-				(font
-					(size 1.27 1.27)
-				)
-			)
-		)
-		(property "LCSC PN" "C72334"
-			(at 247.65 58.42 0)
-			(hide yes)
-			(show_name no)
-			(do_not_autoplace no)
-			(effects
-				(font
-					(size 1.27 1.27)
-				)
-			)
-		)
-		(pin "2"
-		)
-		(pin "1"
-		)
-		(pin "3"
-		)
-		(instances
-			(project "ratgdo-esp32c6-mini"
-				(path "/d526daf5-1a87-4c4a-b8db-6120ccadc008"
-					(reference "J2")
-					(unit 1)
-				)
-			)
-		)
 	)
 	(symbol
@@
 					(unit 1)
 				)
+			)
+		)
+	)
+	(symbol
+		(lib_id "Connector_Generic:Conn_01x03")
+		(at 247.65 58.42 0)
+		(unit 1)
+		(body_style 1)
+		(exclude_from_sim no)
+		(in_bom yes)
+		(on_board yes)
+		(in_pos_files yes)
+		(dnp no)
+		(property "Reference" "J2"
+			(at 246.38 50.038 0)
+			(show_name no)
+			(do_not_autoplace no)
+			(effects
+				(font
+					(size 1.27 1.27)
+				)
+				(justify left)
+			)
+		)
+		(property "Value" "Conn_01x03"
+			(at 242.062 52.324 0)
+			(show_name no)
+			(do_not_autoplace no)
+			(effects
+				(font
+					(size 1.27 1.27)
+				)
+				(justify left)
+			)
+		)
+		(property "Footprint" "LCSC:CONN-SMD_3P-P2.50_HX-2.54-3P-WT"
+			(at 247.65 58.42 0)
+			(hide yes)
+			(show_name no)
+			(do_not_autoplace no)
+			(effects
+				(font
+					(size 1.27 1.27)
+				)
+			)
+		)
+		(property "Datasheet" ""
+			(at 247.65 58.42 0)
+			(hide yes)
+			(show_name no)
+			(do_not_autoplace no)
+			(effects
+				(font
+					(size 1.27 1.27)
+				)
+			)
+		)
+		(property "Description" "Generic connector, single row, 01x03, script generated (kicad-library-utils/schlib/autogen/connector/)"
+			(at 247.65 58.42 0)
+			(hide yes)
+			(show_name no)
+			(do_not_autoplace no)
+			(effects
+				(font
+					(size 1.27 1.27)
+				)
+			)
+		)
+		(property "LCSC PN" "C5142099"
+			(at 247.65 58.42 0)
+			(hide yes)
+			(show_name no)
+			(do_not_autoplace no)
+			(effects
+				(font
+					(size 1.27 1.27)
+				)
+			)
+		)
+		(pin "3"
+		)
+		(pin "2"
+		)
+		(pin "1"
+		)
+		(instances
+			(project "ratgdo-esp32c6-mini"
+				(path "/d526daf5-1a87-4c4a-b8db-6120ccadc008"
+					(reference "J2")
+					(unit 1)
+				)

Commit message: add dedicated power input
Parts:
- added J2: Conn_01x02, LCSC:CONN-SMD_2P-P2.54-XH2.54-WT, symbol Connector_Generic:Conn_01x02
- renumbered J2 to J3
Connections:
- net +5V: now also J2.1 (Pin_1)
- net GND: now also J2.2 (Pin_2)
Other:
- moved on the sheet: C1, C2, C3, C4, D1, D2, R10, R11, R14, R9, SW1, SW2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

Commit message: change R&C to 0402 size
Parts:
- C1, C3, C4: footprint Capacitor_SMD:C_0805_2012Metric -> Capacitor_SMD:C_0402_1005Metric; LCSC PN C116352 -> C52923
- C2: footprint Capacitor_SMD:C_0805_2012Metric -> Capacitor_SMD:C_0402_1005Metric; LCSC PN C1710 -> C15195
- R1, R2: footprint Resistor_SMD:R_0805_2012Metric -> Resistor_SMD:R_0402_1005Metric; LCSC PN C27834 -> C105872
- R10, R6, R9: footprint Resistor_SMD:R_0805_2012Metric -> Resistor_SMD:R_0402_1005Metric; LCSC PN C17513 -> C106235
- R11, R12, R13, R14, R5, R7, R8: footprint Resistor_SMD:R_0805_2012Metric -> Resistor_SMD:R_0402_1005Metric; LCSC PN C17414 -> C60490
- R3, R4: footprint Resistor_SMD:R_0805_2012Metric -> Resistor_SMD:R_0402_1005Metric; LCSC PN C25295 -> C114765
Changed lines of the file:
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@@
 			)
 		)
-		(property "Footprint" "Resistor_SMD:R_0805_2012Metric"
+		(property "Footprint" "Resistor_SMD:R_0402_1005Metric"
 			(at 99.06 136.398 90)
 			(hide yes)
@@
 			)
 		)
-		(property "LCSC PN" "C25295"
+		(property "LCSC PN" "C114765"
 			(at 99.06 134.62 90)
 			(hide yes)
@@
 			)
 		)
-		(property "Footprint" "Resistor_SMD:R_0805_2012Metric"
+		(property "Footprint" "Resistor_SMD:R_0402_1005Metric"
 			(at 193.548 55.88 90)
 			(hide yes)
@@
 			)
 		)
-		(property "LCSC PN" "C17414"
+		(property "LCSC PN" "C60490"
 			(at 191.77 55.88 0)
 			(hide yes)
@@
 			)
 		)
-		(property "Footprint" "Resistor_SMD:R_0805_2012Metric"
+		(property "Footprint" "Resistor_SMD:R_0402_1005Metric"
 			(at 155.702 33.02 90)
 			(hide yes)
@@
 			)
 		)
-		(property "LCSC PN" "C17414"
+		(property "LCSC PN" "C60490"
 			(at 157.48 33.02 0)
 			(hide yes)
@@
 			)
 		)
-		(property "Footprint" "Resistor_SMD:R_0805_2012Metric"
+		(property "Footprint" "Resistor_SMD:R_0402_1005Metric"
 			(at 60.96 36.068 90)
 			(hide yes)
@@
 			)
 		)
-		(property "LCSC PN" "C27834"
+		(property "LCSC PN" "C105872"
 			(at 60.96 34.29 90)
 			(hide yes)
@@
 			)
 		)
-		(property "Footprint" "Capacitor_SMD:C_0805_2012Metric"
+		(property "Footprint" "Capacitor_SMD:C_0402_1005Metric"
 			(at 208.5848 125.73 0)
 			(hide yes)
@@
 			)
 		)
-		(property "LCSC PN" "C1710"
+		(property "LCSC PN" "C15195"
 			(at 209.55 121.92 0)
 			(hide yes)
@@
 			)
 		)
-		(property "Footprint" "Capacitor_SMD:C_0805_2012Metric"
+		(property "Footprint" "Capacitor_SMD:C_0402_1005Metric"
 			(at 181.9148 125.73 0)
 			(hide yes)
@@
 			)
 		)
-		(property "LCSC PN" "C116352"
+		(property "LCSC PN" "C52923"
 			(at 182.88 121.92 0)
 			(hide yes)
@@
 			)
 		)
-		(property "Footprint" "Resistor_SMD:R_0805_2012Metric"
+		(property "Footprint" "Resistor_SMD:R_0402_1005Metric"
 			(at 230.632 31.75 90)
 			(hide yes)
@@
 			)
 		)
-		(property "LCSC PN" "C17414"
+		(property "LCSC PN" "C60490"
 			(at 232.41 31.75 0)
 			(hide yes)
@@
 			)
 		)
-		(property "Footprint" "Resistor_SMD:R_0805_2012Metric"
+		(property "Footprint" "Resistor_SMD:R_0402_1005Metric"
 			(at 99.06 138.938 90)
 			(hide yes)
@@
 			)
 		)
-		(property "LCSC PN" "C25295"
+		(property "LCSC PN" "C114765"
 			(at 99.06 137.16 90)
 			(hide yes)
@@
 			)
 		)
-		(property "Footprint" "Resistor_SMD:R_0805_2012Metric"
+		(property "Footprint" "Resistor_SMD:R_0402_1005Metric"
 			(at 184.15 46.482 90)
 			(hide yes)
@@
 			)
 		)
-		(property "LCSC PN" "C17414"
+		(property "LCSC PN" "C60490"
 			(at 184.15 48.26 90)
 			(hide yes)
@@
 			)
 		)
-		(property "Footprint" "Capacitor_SMD:C_0805_2012Metric"
+		(property "Footprint" "Capacitor_SMD:C_0402_1005Metric"
 			(at 244.8052 121.92 0)
 			(hide yes)
@@
 			)
 		)
-		(property "LCSC PN" "C116352"
+		(property "LCSC PN" "C52923"
 			(at 243.84 118.11 0)
 			(hide yes)
@@
 			)
 		)
-		(property "Footprint" "Resistor_SMD:R_0805_2012Metric"
+		(property "Footprint" "Resistor_SMD:R_0402_1005Metric"
 			(at 242.062 107.95 90)
 			(hide yes)
@@
 			)
 		)
-		(property "LCSC PN" "C17414"
+		(property "LCSC PN" "C60490"
 			(at 243.84 107.95 0)
 			(hide yes)
@@
 			)
 		)
-		(property "Footprint" "Resistor_SMD:R_0805_2012Metric"
+		(property "Footprint" "Resistor_SMD:R_0402_1005Metric"
 			(at 163.83 26.162 90)
 			(hide yes)
@@
 			)
 		)
-		(property "LCSC PN" "C17513"
+		(property "LCSC PN" "C106235"
 			(at 163.83 27.94 90)
 			(hide yes)
@@
 			)
 		)
-		(property "Footprint" "Resistor_SMD:R_0805_2012Metric"
+		(property "Footprint" "Resistor_SMD:R_0402_1005Metric"
 			(at 60.96 38.608 90)
 			(hide yes)
@@
 			)
 		)
-		(property "LCSC PN" "C27834"
+		(property "LCSC PN" "C105872"
 			(at 60.96 36.83 90)
 			(hide yes)
@@
 			)
 		)
-		(property "Footprint" "Capacitor_SMD:C_0805_2012Metric"
+		(property "Footprint" "Capacitor_SMD:C_0402_1005Metric"
 			(at 214.9348 125.73 0)
 			(hide yes)
@@
 			)
 		)
-		(property "LCSC PN" "C116352"
+		(property "LCSC PN" "C52923"
 			(at 215.9 121.92 0)
 			(hide yes)
@@
 			)
 		)
-		(property "Footprint" "Resistor_SMD:R_0805_2012Metric"
+		(property "Footprint" "Resistor_SMD:R_0402_1005Metric"
 			(at 229.362 107.95 90)
 			(hide yes)
@@
 			)
 		)
-		(property "LCSC PN" "C17414"
+		(property "LCSC PN" "C60490"
 			(at 231.14 107.95 0)
 			(hide yes)
@@
 			)
 		)
-		(property "Footprint" "Resistor_SMD:R_0805_2012Metric"
+		(property "Footprint" "Resistor_SMD:R_0402_1005Metric"
 			(at 210.82 149.098 90)
 			(hide yes)
@@
 			)
 		)
-		(property "LCSC PN" "C17513"
+		(property "LCSC PN" "C106235"
 			(at 210.82 147.32 90)
 			(hide yes)
@@
 			)
 		)
-		(property "Footprint" "Resistor_SMD:R_0805_2012Metric"
+		(property "Footprint" "Resistor_SMD:R_0402_1005Metric"
 			(at 210.82 150.622 90)
 			(hide yes)
@@
 			)
 		)
-		(property "LCSC PN" "C17513"
+		(property "LCSC PN" "C106235"
 			(at 210.82 152.4 90)
 			(hide yes)
@@
 			)
 		)
-		(property "Footprint" "Resistor_SMD:R_0805_2012Metric"
+		(property "Footprint" "Resistor_SMD:R_0402_1005Metric"
 			(at 238.76 24.892 90)
 			(hide yes)
@@
 			)
 		)
-		(property "LCSC PN" "C17414"
+		(property "LCSC PN" "C60490"
 			(at 238.76 26.67 90)
 			(hide yes)

Commit message: layout components
Parts:
- J1: value USB_C_Receptacle_USB2.0_14P -> USB_C_2.0
- U2: value ESP32-C6-MINI-1/U -> ESP32-C6-MINI
Changed lines of the file:
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@@
 			)
 		)
-		(property "Value" "ESP32-C6-MINI-1/U"
+		(property "Value" "ESP32-C6-MINI"
 			(at 65.6433 121.92 0)
 			(show_name no)
@@
 			)
 		)
-		(property "Value" "USB_C_Receptacle_USB2.0_14P"
+		(property "Value" "USB_C_2.0"
 			(at 36.83 24.13 0)
 			(show_name no)

Commit message: wiring & cut
Parts:
- removed J2: Conn_01x02, LCSC:CONN-SMD_2P-P2.54-XH2.54-WT, symbol Connector_Generic:Conn_01x02
- removed J3: Conn_01x03, LCSC:CONN-SMD_3P-P2.50_HX-2.54-3P-WT, symbol Connector_Generic:Conn_01x03
- added J2: Conn_01x02, symbol Connector_Generic_Shielded:Conn_01x02_Shielded
- added J3: Conn_01x03, symbol Connector_Generic_Shielded:Conn_01x03_Shielded
Connections:
- net +5V: now also J2.1 (Pin_1)
- net BLK/OBST: now also J3.1 (Pin_1)
- net GND: now also J2.2 (Pin_2), J2.SH (Shield), J3.3 (Pin_3), J3.SH (Shield)
- net RED/CTRL: now also J3.2 (Pin_2)
