File: ratgdo-esp32c6-mini.kicad_pcb (KiCad board)
At the start: 2 copper layers, 38.8 x 27.5 mm, 30 parts, among them J1 USB_C_2.0, J2 Conn_01x02, J3 Conn_01x03, Q1 2N7002, Q2 AO3400A, SW1 RESET, SW2 BOOTSEL, U1 USBLC6-2SC6, U2 ESP32-C6-MINI, U3 RS3236-3.3YF5

Commit message: move via
Routing:
- net +5V: track 25.3 -> 23.8 mm
- net BLK/OBST: track 3.65 -> 2.45 mm
- net RED/CTRL: track 7.53 -> 6.44 mm
Changed lines of the file:
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@@
-	)
-	(segment
-		(start 166.23 99.98)
-		(end 166.75 100.5)
-		(width 0.2)
-		(layer "F.Cu")
-		(net "GND")
 	)
 	(segment
@@
 	)
 	(segment
-		(start 166 99.98)
-		(end 166.23 99.98)
-		(width 0.2)
-		(layer "F.Cu")
-		(net "GND")
-	)
-	(segment
 		(start 153.5625 98.5625)
 		(end 152.5 97.5)
@@
 	)
 	(via
-		(at 166.75 100.5)
+		(at 166 99.98)
 		(size 0.6)
 		(drill 0.3)
@@
 	)
 	(segment
+		(start 166.98 100.27)
+		(end 167.23 100.27)
+		(width 0.2)
+		(layer "B.Cu")
+		(net "GND")
+	)
+	(segment
 		(start 159.975 98.575)
 		(end 159.975 96.6)
@@
 	)
 	(segment
-		(start 167.23 100.27)
-		(end 166.98 100.27)
-		(width 0.2)
-		(layer "B.Cu")
-		(net "GND")
-	)
-	(segment
 		(start 155.75 94.75)
 		(end 155.9 94.75)
@@
 	)
 	(segment
+		(start 166 99.98)
+		(end 166.69 99.98)
+		(width 0.2)
+		(layer "B.Cu")
+		(net "GND")
+	)
+	(segment
+		(start 166.69 99.98)
+		(end 166.98 100.27)
+		(width 0.2)
+		(layer "B.Cu")
+		(net "GND")
+	)
+	(segment
 		(start 159.975 96.6)
 		(end 159.975 94.625)
@@
 	)
 	(segment
-		(start 166.98 100.27)
-		(end 166.75 100.5)
-		(width 0.2)
-		(layer "B.Cu")
-		(net "GND")
-	)
-	(segment
 		(start 156.025 94.625)
 		(end 158 94.625)
@@
 	)
 	(segment
-		(start 166.6175 97.45)
-		(end 167.95 97.45)
-		(width 0.2)
-		(layer "F.Cu")
-		(net "+5V")
-	)
-	(segment
 		(start 158 103.024999)
 		(end 158 102.3625)
@@
 		(net "+5V")
 	)
-	(segment
-		(start 167.95 97.45)
-		(end 168 97.5)
-		(width 0.2)
-		(layer "F.Cu")
-		(net "+5V")
-	)
-	(via
-		(at 168 97.5)
+	(via
+		(at 166.6175 97.45)
 		(size 0.6)
 		(drill 0.3)
@@
 	)
 	(segment
-		(start 167.77 97.73)
-		(end 168 97.5)
-		(width 0.2)
-		(layer "B.Cu")
-		(net "+5V")
-	)
-	(segment
 		(start 157.669132 103.329104)
 		(end 157.669132 103.330868)
@@
 	)
 	(segment
+		(start 166.95 97.45)
+		(end 167.23 97.73)
+		(width 0.2)
+		(layer "B.Cu")
+		(net "+5V")
+	)
+	(segment
 		(start 155.6 104.4)
 		(end 155.6 105)
@@
 	)
 	(segment
-		(start 167.23 97.73)
-		(end 167.77 97.73)
+		(start 166.6175 97.45)
+		(end 166.95 97.45)
 		(width 0.2)
 		(layer "B.Cu")
@@
 	)
 	(segment
-		(start 150.0525 102.45)
+		(start 148.35 101.5)
 		(end 149.1025 101.5)
 		(width 0.2)
@@
 	)
 	(segment
+		(start 148.1 101.25)
+		(end 148.35 101.5)
+		(width 0.2)
+		(layer "F.Cu")
+		(net "BLK{slash}OBST")
+	)
+	(segment
 		(start 149.1025 101.5)
-		(end 147.5 101.5)
+		(end 150.0525 102.45)
 		(width 0.2)
 		(layer "F.Cu")
@@
 	)
 	(via
-		(at 147.5 101.5)
-		(size 0.6)
-		(drill 0.3)
-		(layers "F.Cu" "B.Cu")
-		(net "BLK{slash}OBST")
-	)
-	(segment
-		(start 147.85 101.5)
-		(end 148.1 101.25)
-		(width 0.2)
-		(layer "B.Cu")
-		(net "BLK{slash}OBST")
-	)
-	(segment
-		(start 147.5 101.5)
-		(end 147.85 101.5)
-		(width 0.2)
-		(layer "B.Cu")
+		(at 148.1 101.25)
+		(size 0.6)
+		(drill 0.3)
+		(layers "F.Cu" "B.Cu")
 		(net "BLK{slash}OBST")
 	)
@@
 	)
 	(segment
-		(start 148.175 99)
-		(end 147.5 99)
+		(start 148.175 98.825)
+		(end 148.175 99)
 		(width 0.2)
 		(layer "F.Cu")
@@
 	)
 	(segment
+		(start 148.175 99)
+		(end 149.125 99.95)
+		(width 0.2)
+		(layer "F.Cu")
+		(net "RED{slash}CTRL")
+	)
+	(segment
+		(start 148.1 98.75)
+		(end 148.175 98.825)
+		(width 0.2)
+		(layer "F.Cu")
+		(net "RED{slash}CTRL")
+	)
+	(segment
 		(start 149.5 96.49)
 		(end 148.88 97.11)
@@
 		(net "RED{slash}CTRL")
 	)
-	(segment
-		(start 149.125 99.95)
-		(end 148.175 99)
-		(width 0.2)
-		(layer "F.Cu")
+	(via
+		(at 148.1 98.75)
+		(size 0.6)
+		(drill 0.3)
+		(layers "F.Cu" "B.Cu")
 		(net "RED{slash}CTRL")
 	)
-	(via
-		(at 147.5 99)
-		(size 0.6)
-		(drill 0.3)
-		(layers "F.Cu" "B.Cu")
-		(net "RED{slash}CTRL")
-	)
-	(segment
-		(start 147.85 99)
-		(end 148.1 98.75)
-		(width 0.2)
-		(layer "B.Cu")
-		(net "RED{slash}CTRL")
-	)
-	(segment
-		(start 147.5 99)
-		(end 147.85 99)
-		(width 0.2)
-		(layer "B.Cu")
-		(net "RED{slash}CTRL")
-	)
